File: Sofle_Wireless/PCB/SofleKeyboard.kicad_pcb (KiCad board)
At the start: 2 copper layers, 145.1 x 115.7 mm, 139 parts, among them J1 Conn_01x05, J2 Conn_01x02, SW1 SW1, SW10 SW10, SW11 SW11, SW12 SW12, SW13 SW13, SW14 SW14, SW15 SW15, SW16 SW16, SW17 SW17, SW18 SW18, SW19 SW19, SW2 SW2, SW20 SW20, SW21 SW21, SW22 SW22, SW23 SW23, SW24 SW24, SW25 SW19, SW26 SW26, SW27 SW27, SW28 SW28, SW29 SW29, SW3 SW3, SW30 SW30, SW4 SW4, SW5 SW5, SW6 SW6, SW7 SW7, SW8 SW8, SW9 SW9, U1 NICE!NANO

Commit message: Exploration of multiple sheet for Schematic
Parts:
- removed JP_ENC_LA1, JP_ENC_LB1, JP_E_L1, JP_E_L10, JP_E_L11, JP_E_L12, JP_E_L2, JP_E_L3, JP_E_L4, JP_E_L5, JP_E_L6, JP_E_L7, JP_E_L8, JP_E_L9, JP_LCD_L1, JP_LCD_L2, JP_LCD_L4, JP_LCD_L5: Jumper_NO_Small, Mechanical_Switches:SolderJumper-2_P1.3mm_Open_TrianglePad1.0x1.5mm_E
- removed JP_ENC_RA1, JP_ENC_RB1, JP_E_R1, JP_E_R10, JP_E_R11, JP_E_R12, JP_E_R2, JP_E_R3, JP_E_R4, JP_E_R5, JP_E_R6, JP_E_R7, JP_E_R8, JP_E_R9, JP_LCD_R1, JP_LCD_R2, JP_LCD_R4, JP_LCD_R5: Jumper_NO_Small, Mechanical_Switches:SolderJumper-2_P1.3mm_Open_TrianglePad1.0x1.5mm_E_Reverse
- removed JP_I_L1, JP_I_L10, JP_I_L11, JP_I_L12, JP_I_L2, JP_I_L3, JP_I_L4, JP_I_L5, JP_I_L6, JP_I_L7, JP_I_L8, JP_I_L9: Jumper_NO_Small, Mechanical_Switches:SolderJumper-2_P1.3mm_Open_TrianglePad1.0x1.5mm_I
- removed JP_I_R1, JP_I_R10, JP_I_R11, JP_I_R12, JP_I_R2, JP_I_R3, JP_I_R4, JP_I_R5, JP_I_R6, JP_I_R7, JP_I_R8, JP_I_R9: Jumper_NO_Small, Mechanical_Switches:SolderJumper-2_P1.3mm_Open_TrianglePad1.0x1.5mm_I_Reverse
- added D36: LED_SK6812MINI, RGB_LED:SK6812_Mini-E_DualSide, F.Cu at (499.8, 130.0)
- added D37: LED_SK6812MINI, RGB_LED:SK6812_Mini-E_DualSide, F.Cu at (499.8, 134.5)
- added D38: LED_SK6812MINI, RGB_LED:SK6812_Mini-E_DualSide, F.Cu at (499.8, 139.0)
- added D39: LED_SK6812MINI, RGB_LED:SK6812_Mini-E_DualSide, F.Cu at (499.8, 143.5)
- added D40: LED_SK6812MINI, RGB_LED:SK6812_Mini-E_DualSide, F.Cu at (499.8, 148.0)
- added D41: D, Mechanical_Switches:Diode_SOD-123(dual side), F.Cu at (364.9, 45.6)
- added D42: D, Mechanical_Switches:Diode_SOD-123(dual side), F.Cu at (364.9, 65.8)
- added D43: D, Mechanical_Switches:Diode_SOD-123(dual side), F.Cu at (364.9, 85.9)
- added D44: D, Mechanical_Switches:Diode_SOD-123(dual side), F.Cu at (364.9, 106.1)
- added D45: D, Mechanical_Switches:Diode_SOD-123(dual side), F.Cu at (364.9, 126.2)
- added D46: D, Mechanical_Switches:Diode_SOD-123(dual side), F.Cu at (364.9, 146.4)
- added D47: D, Mechanical_Switches:Diode_SOD-123(dual side), F.Cu at (364.9, 166.5)
- added D48: D, Mechanical_Switches:Diode_SOD-123(dual side), F.Cu at (364.9, 186.7)
- added D49: D, Mechanical_Switches:Diode_SOD-123(dual side), F.Cu at (364.9, 206.8)
- added D50: D, Mechanical_Switches:Diode_SOD-123(dual side), F.Cu at (385.1, 45.6)
- added D51: D, Mechanical_Switches:Diode_SOD-123(dual side), F.Cu at (385.1, 65.8)
- added D52: D, Mechanical_Switches:Diode_SOD-123(dual side), F.Cu at (385.1, 85.9)
- added D53: D, Mechanical_Switches:Diode_SOD-123(dual side), F.Cu at (385.1, 106.1)
- added D54: D, Mechanical_Switches:Diode_SOD-123(dual side), F.Cu at (385.1, 126.2)
- added D55: D, Mechanical_Switches:Diode_SOD-123(dual side), F.Cu at (385.1, 146.4)
- added D56: D, Mechanical_Switches:Diode_SOD-123(dual side), F.Cu at (385.1, 166.5)
- added D57: D, Mechanical_Switches:Diode_SOD-123(dual side), F.Cu at (385.1, 186.7)
- added D58: D, Mechanical_Switches:Diode_SOD-123(dual side), F.Cu at (385.1, 206.8)
- added D59: D, Mechanical_Switches:Diode_SOD-123(dual side), F.Cu at (405.2, 45.6)
- added D60: D, Mechanical_Switches:Diode_SOD-123(dual side), F.Cu at (405.2, 65.8)
- added D61: D, Mechanical_Switches:Diode_SOD-123(dual side), F.Cu at (405.2, 85.9)
- added D62: D, Mechanical_Switches:Diode_SOD-123(dual side), F.Cu at (405.2, 106.1)
- added D63: D, Mechanical_Switches:Diode_SOD-123(dual side), F.Cu at (405.2, 126.2)
- added D64: D, Mechanical_Switches:Diode_SOD-123(dual side), F.Cu at (405.2, 146.4)
- added D65: D, Mechanical_Switches:Diode_SOD-123(dual side), F.Cu at (405.2, 166.5)
- added D66: D, Mechanical_Switches:Diode_SOD-123(dual side), F.Cu at (405.2, 186.7)
- added D67: D, Mechanical_Switches:Diode_SOD-123(dual side), F.Cu at (405.2, 206.8)
- added D68: D, Mechanical_Switches:Diode_SOD-123(dual side), F.Cu at (425.4, 45.6)
- added D69: D, Mechanical_Switches:Diode_SOD-123(dual side), F.Cu at (425.4, 65.8)
- added D70: D, Mechanical_Switches:Diode_SOD-123(dual side), F.Cu at (425.4, 85.9)
- added EC2: Rotary_Encoder_Switch, Mechanical_Switches:RotaryEncoder_Alps_EC12E-Switch_Vertical_H20mm, F.Cu at (504.9, 158.9)
- added J3: Conn_01x05, Mechanical_Switches:NICE!VIEW, F.Cu at (503.4, 69.6)
- added J4: Conn_01x02, Mechanical_Switches:JST_PH_S2B-PH-SM4-TB_1x02-1MP_P2.00mm_Horizontal_DualSide, F.Cu at (501.0, 181.0)
- added PWR_SW2: Switch, Mechanical_Switches:SLW-1276864-4A-D, F.Cu at (502.8, 171.4)
- added R3: R, Mechanical_Switches:R_0805_2012Metric_Pad1.20x1.40mm_HandSolder_dualside, F.Cu at (508.5, 181.5)
- added R4: R, Mechanical_Switches:R_0805_2012Metric_Pad1.20x1.40mm_HandSolder_dualside, F.Cu at (508.5, 184.4)
- added RSW2: SW_RST, Mechanical_Switches:ResetSW_DualSide, F.Cu at (510.9, 177.7)
- added SW31: SW1, Mechanical_Switches:SW_MXHS_CHOCV1V2HS_1U, F.Cu at (425.4, 106.1)
- added SW32: SW7, Mechanical_Switches:SW_MXHS_CHOCV1V2HS_1U, F.Cu at (425.4, 126.2)
- added SW33: SW13, Mechanical_Switches:SW_MXHS_CHOCV1V2HS_1U, F.Cu at (425.4, 146.4)
- added SW34: SW19, Mechanical_Switches:SW_MXHS_CHOCV1V2HS_1U, F.Cu at (425.4, 166.5)
- added SW35: SW19, Mechanical_Switches:SW_MXHS_CHOCV1V2HS_1U, F.Cu at (425.4, 186.7)
- added SW36: SW2, Mechanical_Switches:SW_MXHS_CHOCV1V2HS_1U, F.Cu at (425.4, 206.8)
- added SW37: SW8, Mechanical_Switches:SW_MXHS_CHOCV1V2HS_1U, F.Cu at (445.5, 45.6)
- added SW38: SW14, Mechanical_Switches:SW_MXHS_CHOCV1V2HS_1U, F.Cu at (445.5, 65.8)
- added SW39: SW20, Mechanical_Switches:SW_MXHS_CHOCV1V2HS_1U, F.Cu at (445.5, 85.9)
- added SW40: SW26, Mechanical_Switches:SW_MXHS_CHOCV1V2HS_1.5U, F.Cu at (510.7, 117.8)
- added SW41: SW3, Mechanical_Switches:SW_MXHS_CHOCV1V2HS_1U, F.Cu at (445.5, 106.1)
- added SW42: SW9, Mechanical_Switches:SW_MXHS_CHOCV1V2HS_1U, F.Cu at (445.5, 126.2)
- added SW43: SW15, Mechanical_Switches:SW_MXHS_CHOCV1V2HS_1U, F.Cu at (445.5, 146.4)
- added SW44: SW21, Mechanical_Switches:SW_MXHS_CHOCV1V2HS_1U, F.Cu at (445.5, 166.5)
- added SW45: SW27, Mechanical_Switches:SW_MXHS_CHOCV1V2HS_1U, F.Cu at (445.5, 186.7)
- added SW46: SW4, Mechanical_Switches:SW_MXHS_CHOCV1V2HS_1U, F.Cu at (445.5, 206.8)
- added SW47: SW10, Mechanical_Switches:SW_MXHS_CHOCV1V2HS_1U, F.Cu at (465.6, 45.6)
- added SW48: SW16, Mechanical_Switches:SW_MXHS_CHOCV1V2HS_1U, F.Cu at (465.6, 65.8)
- added SW49: SW22, Mechanical_Switches:SW_MXHS_CHOCV1V2HS_1U, F.Cu at (465.6, 85.9)
- added SW50: SW28, Mechanical_Switches:SW_MXHS_CHOCV1V2HS_1U, F.Cu at (465.6, 106.1)
- added SW51: SW5, Mechanical_Switches:SW_MXHS_CHOCV1V2HS_1U, F.Cu at (465.6, 126.2)
- added SW52: SW11, Mechanical_Switches:SW_MXHS_CHOCV1V2HS_1U, F.Cu at (465.6, 146.4)
- added SW53: SW17, Mechanical_Switches:SW_MXHS_CHOCV1V2HS_1U, F.Cu at (465.6, 166.5)
- added SW54: SW23, Mechanical_Switches:SW_MXHS_CHOCV1V2HS_1U, F.Cu at (465.6, 186.7)
- added SW55: SW29, Mechanical_Switches:SW_MXHS_CHOCV1V2HS_1U, F.Cu at (465.6, 206.8)
- added SW56: SW6, Mechanical_Switches:SW_MXHS_CHOCV1V2HS_1U, F.Cu at (485.8, 45.6)
- added SW57: SW12, Mechanical_Switches:SW_MXHS_CHOCV1V2HS_1U, F.Cu at (485.8, 65.8)
- added SW58: SW18, Mechanical_Switches:SW_MXHS_CHOCV1V2HS_1U, F.Cu at (485.8, 85.9)
- added SW59: SW24, Mechanical_Switches:SW_MXHS_CHOCV1V2HS_1U, F.Cu at (485.8, 106.1)
- added SW60: SW30, Mechanical_Switches:SW_MXHS_CHOCV1V2HS_1U, F.Cu at (485.8, 126.2)
- added TH10: HOLE, MountingHole:MountingHole_2.2mm_M2, F.Cu at (512.6, 136.8)
- added TH11: HOLE, MountingHole:MountingHole_2.2mm_M2, F.Cu at (518.5, 130.9)
- added TH12: HOLE, MountingHole:MountingHole_2.2mm_M2, F.Cu at (518.5, 136.8)
- added TH7: HOLE, MountingHole:MountingHole_2.2mm_M2, F.Cu at (506.6, 130.9)
- added TH8: HOLE, MountingHole:MountingHole_2.2mm_M2, F.Cu at (506.6, 136.8)
- added TH9: HOLE, MountingHole:MountingHole_2.2mm_M2, F.Cu at (512.6, 130.9)
- added U2: NICE!NANO, Mechanical_Switches:NICE!NANO, F.Cu at (505.3, 90.7)
Connections:
- EC1 pad A: Net-(EC1-PadA) -> ENCA
- EC1 pad B: Net-(EC1-PadB) -> ENCB
- J1 pad 1: Net-(J1-Pin_1) -> SDA
- J1 pad 2: Net-(J1-Pin_2) -> SCL
- J1 pad 4: Net-(J1-Pin_4) -> GND
- J1 pad 5: Net-(J1-Pin_5) -> CS
- U1 pad 1: Net-(U1-EXT1) -> BATT+
- U1 pad 10: Net-(U1-EXT10) -> col3
- U1 pad 11: Net-(U1-EXT11) -> col4
- U1 pad 12: Net-(U1-EXT12) -> col5
- U1 pad 13: Net-(U1-INT12) -> row4
- U1 pad 14: Net-(U1-INT11) -> row3
- U1 pad 15: Net-(U1-INT10) -> row2
- U1 pad 16: Net-(U1-INT9) -> row1
- U1 pad 17: Net-(U1-INT8) -> row0
- U1 pad 18: Net-(U1-INT7) -> unconnected-(U1-INT7-Pad18)
- U1 pad 19: Net-(U1-INT6) -> SCL
- U1 pad 2: Net-(U1-EXT2) -> GND
- U1 pad 20: Net-(U1-INT5) -> SDA
- U1 pad 21: Net-(U1-INT4) -> GND
- U1 pad 22: Net-(U1-INT3) -> GND
- U1 pad 23: Net-(U1-INT2) -> LED
- U1 pad 24: Net-(U1-INT1) -> CS
- U1 pad 3: Net-(U1-EXT3) -> RESET
- U1 pad 4: Net-(U1-EXT4) -> VCC
- U1 pad 5: Net-(U1-EXT5) -> ENCA
- U1 pad 6: Net-(U1-EXT6) -> ENCB
- U1 pad 7: Net-(U1-EXT7) -> col0
- U1 pad 8: Net-(U1-EXT8) -> col1
- U1 pad 9: Net-(U1-EXT9) -> col2
Routing:
- net col0: track 286.0 -> 0.00 mm, vias 22 -> 0
- net col1: track 276.4 -> 0.00 mm, vias 19 -> 0
- net col2: track 254.6 -> 0.00 mm, vias 17 -> 0
- net col3: track 240.9 -> 0.00 mm, vias 15 -> 0
- net col4: track 210.4 -> 0.00 mm, vias 13 -> 0
- net row4: track 186.8 -> 0.00 mm, vias 7 -> 0
- net VCC: track 181.5 -> 0.00 mm, vias 8 -> 0
- net row3: track 172.6 -> 0.00 mm, vias 7 -> 0
- net col5: track 171.3 -> 0.00 mm, vias 11 -> 0
- net row0: track 157.5 -> 0.00 mm, vias 7 -> 0
- net row2: track 153.5 -> 0.00 mm, vias 7 -> 0
- net row1: track 142.8 -> 0.00 mm, vias 7 -> 0
- net BATT+: track 82.0 -> 0.00 mm, vias 1 -> 0
- net LED: track 78.0 -> 0.00 mm, vias 4 -> 0
- net CS: track 75.4 -> 0.00 mm, vias 3 -> 0
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- removed copper zone on B.Cu, net GND
- removed copper zone on F.Cu, net GND
